Commit message: Updated ras545_hw3 with gazebo launch

File: urdf/hw3_scara_gazebo.urdf (robot description, URDF)
Before this commit: robot hw3_scara, 8 links, 7 joints
Links:
- added link world
Joints:
- added joint joint0_fixed: type fixed, parent world, child base_link, origin xyz=0 0 0 rpy=0 0 0

File: urdf/hw3_scara_rviz.urdf (robot description, URDF)
Before this commit: robot hw3_scara, 8 links, 7 joints
Links:
- added link world
Joints:
- added joint joint0_fixed: type fixed, parent world, child base_link, origin xyz=0 0 0 rpy=0 0 0
